File: JN5189_pcb_v1/jn5189_pcb_v1.brd (EAGLE design)
At the start: 16.1 x 30 mm, 25 parts, among them Y1 32.768KHz, Y2 32Mhz

Commit message: Add files via upload
Routing:
- net GND: vias 400 -> 417

Commit message: Add files via upload
Parts:
- added 3V3, GND, ISP, RXD, TXD: TPSTP11R, testpad:TP11R
Connections:
- net GND: now also GND.TP
- net PIO5: now also ISP.TP
- net PIO8: now also TXD.TP
- net PIO9: now also RXD.TP
- net VDD: now also 3V3.TP
Routing:
- net VDD: track 23.7 -> 33.3 mm
- net PIO5: track 4.48 -> 8.77 mm
- net PIO8: track 2.97 -> 4.49 mm
- net PIO9: track 2.65 -> 4.16 mm
- net GND: vias 417 -> 418

Commit message: Add files via upload
Routing:
- net GND: track 53.9 -> 52.7 mm, vias 418 -> 419
- net PIO8: track 4.49 -> 4.67 mm, vias 0 -> 1
- net VDD: track 33.3 -> 33.5 mm, vias 2 -> 3
- net PIO9: track 4.16 -> 4.22 mm, vias 0 -> 1
- net PIO5: vias 0 -> 1
Other:
- board text added: "ISP"
- board text added: "RX"
- board text added: "TX"

Commit message: Add files via upload
Routing:
- net GND: vias 419 -> 418
Changed lines of the file:
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@@
 <setting verticaltext="up"/>
 </settings>
-<grid distance="0.127" unitdist="mm" unit="mm" style="lines" multiple="1" display="yes" altdistance="5" altunitdist="mil" altunit="mm"/>
+<grid distance="0.01" unitdist="mm" unit="mm" style="lines" multiple="1" display="yes" altdistance="5" altunitdist="mil" altunit="mm"/>
 <layers>
 <layer number="1" name="Top" color="4" fill="1" visible="yes" active="yes"/>
@@
 <polygon width="0.1524" layer="16" thermals="no">
 <vertex x="0.1778" y="-0.1524"/>
-<vertex x="16.5288" y="-0.1524"/>
-<vertex x="16.5288" y="24.8689"/>
-<vertex x="0.1778" y="24.8689"/>
+<vertex x="16.4488" y="-0.1524"/>
+<vertex x="16.4488" y="24.8989"/>
+<vertex x="0.1778" y="24.8989"/>
 </polygon>
 <contactref element="Y2" pad="2"/>
@@
 <vertex x="9.652" y="7.239"/>
 <vertex x="9.652" y="14.859"/>
-<vertex x="16.637" y="14.859"/>
-<vertex x="16.637" y="24.892"/>
+<vertex x="16.487" y="14.859"/>
+<vertex x="16.487" y="24.892"/>
 <vertex x="0.127" y="24.892"/>
 <vertex x="0.127" y="-0.127"/>
@@
 <via x="4.749671875" y="23.687315625" extent="1-16" drill="0.2" diameter="0.45"/>
 <via x="4.6532625" y="24.1600875" extent="1-16" drill="0.2" diameter="0.45"/>
-<via x="4.752278125" y="24.62988125" extent="1-16" drill="0.2" diameter="0.45"/>
-<via x="3.533959375" y="24.650271875" extent="1-16" drill="0.2" diameter="0.45"/>
+<via x="4.762278125" y="24.70988125" extent="1-16" drill="0.2" diameter="0.45"/>
+<via x="3.503959375" y="24.710271875" extent="1-16" drill="0.2" diameter="0.45"/>
 <via x="3.641009375" y="24.16086875" extent="1-16" drill="0.2" diameter="0.45"/>
 <via x="3.709715625" y="23.695321875" extent="1-16" drill="0.2" diameter="0.45"/>
@@
 <via x="5.01209375" y="18.65866875" extent="1-16" drill="0.2" diameter="0.45"/>
 <via x="5.470946875" y="18.777375" extent="1-16" drill="0.2" diameter="0.45"/>
-<via x="5.752278125" y="24.62988125" extent="1-16" drill="0.2" diameter="0.45"/>
-<via x="6.752278125" y="24.62988125" extent="1-16" drill="0.2" diameter="0.45"/>
-<via x="7.752278125" y="24.62988125" extent="1-16" drill="0.2" diameter="0.45"/>
-<via x="8.752278125" y="24.62988125" extent="1-16" drill="0.2" diameter="0.45"/>
-<via x="9.752278125" y="24.62988125" extent="1-16" drill="0.2" diameter="0.45"/>
-<via x="10.752278125" y="24.62988125" extent="1-16" drill="0.2" diameter="0.45"/>
-<via x="11.752278125" y="24.62988125" extent="1-16" drill="0.2" diameter="0.45"/>
-<via x="12.752278125" y="24.62988125" extent="1-16" drill="0.2" diameter="0.45"/>
-<via x="13.752278125" y="24.62988125" extent="1-16" drill="0.2" diameter="0.45"/>
-<via x="14.752278125" y="24.62988125" extent="1-16" drill="0.2" diameter="0.45"/>
-<via x="15.752278125" y="24.62988125" extent="1-16" drill="0.2" diameter="0.45"/>
+<via x="5.752278125" y="24.70988125" extent="1-16" drill="0.2" diameter="0.45"/>
+<via x="6.752278125" y="24.71988125" extent="1-16" drill="0.2" diameter="0.45"/>
+<via x="7.752278125" y="24.71988125" extent="1-16" drill="0.2" diameter="0.45"/>
+<via x="8.742278125" y="24.71988125" extent="1-16" drill="0.2" diameter="0.45"/>
+<via x="9.752278125" y="24.71988125" extent="1-16" drill="0.2" diameter="0.45"/>
+<via x="10.752278125" y="24.71988125" extent="1-16" drill="0.2" diameter="0.45"/>
+<via x="11.762278125" y="24.70988125" extent="1-16" drill="0.2" diameter="0.45"/>
+<via x="12.742278125" y="24.70988125" extent="1-16" drill="0.2" diameter="0.45"/>
+<via x="13.752278125" y="24.70988125" extent="1-16" drill="0.2" diameter="0.45"/>
+<via x="14.752278125" y="24.70988125" extent="1-16" drill="0.2" diameter="0.45"/>
+<via x="15.742278125" y="24.70988125" extent="1-16" drill="0.2" diameter="0.45"/>
 <via x="5.1612625" y="24.1600875" extent="1-16" drill="0.2" diameter="0.45"/>
 <via x="5.306615625" y="23.705671875" extent="1-16" drill="0.2" diameter="0.45"/>
@@
 <via x="7.752278125" y="19.12988125" extent="1-16" drill="0.2" diameter="0.45"/>
 <via x="7.752278125" y="19.87988125" extent="1-16" drill="0.2" diameter="0.45"/>
-<via x="0.672278125" y="24.62988125" extent="1-16" drill="0.2" diameter="0.45"/>
+<via x="0.662278125" y="24.71988125" extent="1-16" drill="0.2" diameter="0.45"/>
 <via x="0.672278125" y="23.61388125" extent="1-16" drill="0.2" diameter="0.45"/>
 <via x="0.672278125" y="22.59788125" extent="1-16" drill="0.2" diameter="0.45"/>
@@
 <via x="1.601278125" y="3.12488125" extent="1-16" drill="0.2" diameter="0.45"/>
 <contactref element="GND" pad="TP"/>
-<via x="1.772278125" y="24.62988125" extent="1-16" drill="0.2" diameter="0.45"/>
-<via x="3.025959375" y="24.650271875" extent="1-16" drill="0.2" diameter="0.45"/>
-<via x="2.390959375" y="24.650271875" extent="1-16" drill="0.2" diameter="0.45"/>
+<via x="1.137278125" y="24.70988125" extent="1-16" drill="0.2" diameter="0.45"/>
+<via x="3.025959375" y="24.710271875" extent="1-16" drill="0.2" diameter="0.45"/>
 </signal>
 <signal name="VDD1">
